File: sch/fan control.sch (KiCad schematic (older format))
At the start: 64 parts, among them J1 Serial Port, J2 Buttons, J3 Power 5V, J4 ICSP, J5 Light, J6 Motor cois, J7 AC 220v in, K1 DIPxx-1Axx-12x, K2 DIPxx-1Axx-12x, K3 DIPxx-1Axx-12x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

Commit message: housekeeping
Connections:
- wire segments 278 -> 282
Changed lines of the file:
@@
 EESchema Schematic File Version 4
+LIBS:fan control-cache
 EELAYER 26 0
 EELAYER END
@@
 	8050 1300 8050 1500
 Connection ~ 8050 1500
+Wire Wire Line
+	2600 6400 4600 6400
+Wire Wire Line
+	4600 6400 4600 5950
+Wire Wire Line
+	4600 5950 1900 5950
+Wire Wire Line
+	1900 5950 1900 5750
 $EndSCHEMATC
