File: sch/fan control.kicad_pcb (KiCad board)
At the start: 2 copper layers, 94 parts, among them J1 Serial Port, J2 Buttons, J3 Power 5V, J5 STATUS LEDs, J6 Light, J7 Motor cois, J8 AC 220v in, K1 SANYOU_SRD_Form_C, K2 SANYOU_SRD_Form_C, K3 SANYOU_SRD_Form_C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

Commit message: Changed pcb
Parts:
- moved ? 56.4 mm to (96.3, 54.4)
- moved REF** 2.54 mm to (120.4, 118.4)
Routing:
- net Net-(R21-Pad2): track 69.5 -> 126.7 mm
- net (no net): track 124.2 -> 70.6 mm
Changed lines of the file:
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@@
     (thickness 1.6)
     (drawings 1)
-    (tracks 485)
+    (tracks 487)
     (zones 0)
     (modules 94)
@@
   )
   (module different:pad (layer F.Cu)
-    (at 98.298 110.744)
+    (at 96.266 54.356)
     (fp_text reference "" (at 0 0) (layer F.SilkS) hide
       (effects (font (size 1 1) (thickness 0.15)))
@@
   )
   (module Symbol:OSHW-Logo2_7.3x6mm_Copper (layer B.Cu)
-    (at 117.856 118.364 180)
+    (at 120.396 118.364 180)
     (descr "Open Source Hardware Symbol")
     (tags "Logo Symbol OSHW")
@@
   (segment (start 115.824 66.294) (end 118.364 68.834) (width 0.8) (layer F.Cu) (net 0))
   (segment (start 106.426 66.294) (end 115.824 66.294) (width 0.8) (layer F.Cu) (net 0))
-  (segment (start 101.854 54.356) (end 99.314 54.356) (width 0.8) (layer F.Cu) (net 0))
-  (segment (start 99.314 54.356) (end 98.298 55.372) (width 0.8) (layer F.Cu) (net 0))
-  (segment (start 98.298 55.372) (end 98.298 110.744) (width 0.8) (layer F.Cu) (net 0))
+  (segment (start 102.108 54.356) (end 96.266 54.356) (width 0.8) (layer F.Cu) (net 0))
   (segment (start 133.604 66.802) (end 133.604 66.802) (width 0.8) (layer B.Cu) (net 2))
   (segment (start 133.604 66.802) (end 133.604 66.802) (width 0.8) (layer B.Cu) (net 2))
@@
   (segment (start 144.272 101.854) (end 143.764 102.362) (width 0.8) (layer B.Cu) (net 62))
   (segment (start 136.144 112.522) (end 134.366 110.744) (width 0.8) (layer B.Cu) (net 62))
-  (segment (start 134.366 110.744) (end 98.298 110.744) (width 0.8) (layer B.Cu) (net 62))
   (segment (start 110.49 55.626) (end 109.474 55.626) (width 0.8) (layer B.Cu) (net 62))
   (segment (start 109.474 55.626) (end 108.204 54.356) (width 0.8) (layer B.Cu) (net 62))
   (segment (start 108.204 54.356) (end 102.362 54.356) (width 0.8) (layer B.Cu) (net 62))
+  (segment (start 134.366 110.744) (end 100.185773 110.744) (width 0.8) (layer B.Cu) (net 62))
+  (segment (start 100.185773 110.744) (end 98.552 110.744) (width 0.8) (layer B.Cu) (net 62))
+  (segment (start 98.552 110.744) (end 98.298 110.744) (width 0.8) (layer B.Cu) (net 62))
+  (segment (start 98.298 110.744) (end 96.266 108.712) (width 0.8) (layer B.Cu) (net 62))
+  (segment (start 96.266 108.712) (end 96.266 54.356) (width 0.8) (layer B.Cu) (net 62))
   (segment (start 151.892 96.774) (end 151.892 100.584) (width 0.8) (layer B.Cu) (net 63))
   (segment (start 154.94 110.236) (end 146.304 118.872) (width 1) (layer B.Cu) (net 64))

Commit message: PCB changed - new heatsynk
Parts:
- moved REF** 24.4 mm to (160.0, 113.0), turned to 0 degrees
- moved Q10 2.34 mm to (174.5, 119.4)
Routing:
- net Net-(Q10-Pad3): track 25.6 -> 31.3 mm
- net Net-(F1-Pad2): track 62.1 -> 67.0 mm
- net Net-(R22-Pad2): track 33.3 -> 30.9 mm
- net Net-(D12-Pad2): track 29.3 -> 31.4 mm

Commit message: pcb
Routing:
- net (no net): track 70.6 -> 95.0 mm
- net Net-(J7-Pad2): track 26.1 -> 23.6 mm
Changed lines of the file:
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@@
     (thickness 1.6)
     (drawings 1)
-    (tracks 487)
+    (tracks 513)
     (zones 0)
     (modules 94)
@@
   (segment (start 106.426 66.294) (end 115.824 66.294) (width 0.8) (layer F.Cu) (net 0))
   (segment (start 102.108 54.356) (end 96.266 54.356) (width 0.8) (layer F.Cu) (net 0))
+  (segment (start 160.02 112.7379) (end 160.02 113.03) (width 2) (layer B.Cu) (net 0))
+  (segment (start 161.1122 111.6457) (end 160.02 112.7379) (width 2) (layer B.Cu) (net 0))
+  (segment (start 160.02 113.2713) (end 161.2011 114.4524) (width 2) (layer B.Cu) (net 0))
+  (segment (start 160.02 113.2713) (end 160.02 113.03) (width 2) (layer B.Cu) (net 0))
+  (segment (start 158.520001 111.418499) (end 158.520001 111.530001) (width 2) (layer B.Cu) (net 0))
+  (segment (start 158.5341 111.4044) (end 158.520001 111.418499) (width 2) (layer B.Cu) (net 0))
+  (segment (start 160.02 113.03) (end 158.520001 114.529999) (width 2) (layer B.Cu) (net 0))
+  (segment (start 158.520001 114.542699) (end 158.520001 114.529999) (width 2) (layer B.Cu) (net 0))
+  (segment (start 160.02 114.7572) (end 160.02 113.03) (width 2) (layer B.Cu) (net 0))
+  (segment (start 160.02 111.6457) (end 159.8041 111.4298) (width 2) (layer B.Cu) (net 0))
+  (segment (start 160.02 113.03) (end 160.02 111.6457) (width 2) (layer B.Cu) (net 0))
+  (segment (start 158.520001 111.530001) (end 159.8041 111.4298) (width 2) (layer B.Cu) (net 0))
+  (segment (start 160.02 113.03) (end 161.6075 113.03) (width 2) (layer B.Cu) (net 0))
+  (segment (start 157.9626 113.03) (end 157.7721 112.8395) (width 2) (layer B.Cu) (net 0))
+  (segment (start 160.02 113.03) (end 157.7721 112.8395) (width 2) (layer B.Cu) (net 0))
+  (segment (start 183.82 113.03) (end 183.82 113.3223) (width 2) (layer B.Cu) (net 0))
+  (segment (start 183.82 113.3223) (end 184.8104 114.3127) (width 2) (layer B.Cu) (net 0))
+  (segment (start 183.82 113.0175) (end 183.82 113.03) (width 2) (layer B.Cu) (net 0))
+  (segment (start 183.82 113.03) (end 182.2704 113.03) (width 2) (layer B.Cu) (net 0))
+  (segment (start 183.82 111.9253) (end 183.7436 111.8489) (width 2) (layer B.Cu) (net 0))
+  (segment (start 183.82 113.03) (end 183.82 111.9253) (width 2) (layer B.Cu) (net 0))
+  (segment (start 183.7436 111.8489) (end 182.753 111.9124) (width 2) (layer B.Cu) (net 0))
+  (segment (start 183.82 113.03) (end 183.82 114.7062) (width 2) (layer B.Cu) (net 0))
+  (segment (start 183.82 114.7062) (end 183.6805 114.5667) (width 2) (layer B.Cu) (net 0))
+  (segment (start 183.6805 114.5667) (end 183.4896 114.5667) (width 2) (layer B.Cu) (net 0))
+  (segment (start 183.4896 114.5667) (end 182.3974 114.6937) (width 2) (layer B.Cu) (net 0))
+  (segment (start 184.7342 113.03) (end 183.82 113.03) (width 2) (layer B.Cu) (net 0))
   (segment (start 149.606 71.374) (end 145.796 75.184) (width 0.8) (layer B.Cu) (net 1))
   (segment (start 145.796 75.184) (end 143.256 75.184) (width 0.8) (layer B.Cu) (net 1))
@@
   (segment (start 173.408 92.156) (end 186.136 92.156) (width 2) (layer B.Cu) (net 30))
   (segment (start 180.594 87.122) (end 186.182 87.122) (width 2) (layer B.Cu) (net 31))
-  (segment (start 179.07 85.598) (end 180.594 87.122) (width 2) (layer B.Cu) (net 31))
-  (segment (start 173.408 73.36) (end 176.23 73.36) (width 2) (layer B.Cu) (net 31))
-  (segment (start 176.23 73.36) (end 178.054 75.184) (width 2) (layer B.Cu) (net 31))
-  (segment (start 178.054 84.582) (end 180.594 87.122) (width 2) (layer B.Cu) (net 31))
-  (segment (start 178.054 75.184) (end 178.054 84.582) (width 2) (layer B.Cu) (net 31))
+  (segment (start 179.5907 86.1187) (end 180.594 87.122) (width 2) (layer B.Cu) (net 31))
+  (segment (start 179.5907 77.42138) (end 179.5907 86.1187) (width 2) (layer B.Cu) (net 31))
+  (segment (start 175.52932 73.36) (end 179.5907 77.42138) (width 2) (layer B.Cu) (net 31))
+  (segment (start 173.408 73.36) (end 175.52932 73.36) (width 2) (layer B.Cu) (net 31))
   (segment (start 173.408 54.564) (end 176.738 54.564) (width 2) (layer B.Cu) (net 32))
   (segment (start 176.738 54.564) (end 179.07 56.896) (width 2) (layer B.Cu) (net 32))
